Commit message: add spacer scads

File: src/ballbot_description/onshape/ballbot/robot.urdf (robot description, URDF)
Before this commit: robot ballbot, 6 links, 5 joints
Links:
- link wheel_assm__configuration_screwless: geometry collision cylinder length=0.006 radius=0.0069282; collision cylinder length=0.006 radius=0.0069282
- link wheel_assm__configuration_screwless_2: geometry collision cylinder length=0.006 radius=0.0069282; collision cylinder length=0.006 radius=0.0069282
- link wheel_assm__configuration_screwless_3: geometry collision cylinder length=0.006 radius=0.0069282; collision cylinder length=0.006 radius=0.0069282
- link wheel_assm__configuration_screwless_4: geometry collision cylinder length=0.006 radius=0.0069282; collision cylinder length=0.006 radius=0.0069282

Commit message: add screws in visual config

File: src/ballbot_description/onshape/ballbot/robot.urdf (robot description, URDF)
Before this commit: robot ballbot, 6 links, 5 joints
Links:
- removed link still_chassis_assm__configuration_screwless
- removed link wheel_assm__configuration_screwless
- removed link wheel_assm__configuration_screwless_2
- removed link wheel_assm__configuration_screwless_3
- removed link wheel_assm__configuration_screwless_4
- added link still_chassis_assm__configuration_default, mass 1.12003; collision box size=0.006 0.014 0.005; collision box size=0.006 0.014 0.005
- added link wheel_assm__configuration_default, mass 0.0544576; collision cylinder length=0.006 radius=0.0069282; collision cylinder length=0.006 radius=0.0069282
- added link wheel_assm__configuration_default_2, mass 0.0544576; collision cylinder length=0.006 radius=0.0069282; collision cylinder length=0.006 radius=0.0069282
- added link wheel_assm__configuration_default_3, mass 0.0544576; collision cylinder length=0.006 radius=0.0069282; collision cylinder length=0.006 radius=0.0069282
- added link wheel_assm__configuration_default_4, mass 0.0544576; collision cylinder length=0.006 radius=0.0069282; collision cylinder length=0.006 radius=0.0069282
Joints:
- removed joint base_link_to_still_chassis_assm__configuration_screwless
- added joint base_link_to_still_chassis_assm__configuration_default: type fixed, parent base_link, child still_chassis_assm__configuration_default, origin xyz=0 0 0 rpy=0 -0 0, axis 0 0 1, limit effort=10 velocity=10
- joint front_left_wheel_speed: child wheel_assm__configuration_screwless -> wheel_assm__configuration_default; parent still_chassis_assm__configuration_screwless -> still_chassis_assm__configuration_default
- joint front_right_wheel_speed: child wheel_assm__configuration_screwless_2 -> wheel_assm__configuration_default_2; origin xyz=0.0680211 -0.0776141 -0.0305 rpy=-1.5708 0.672397 3.45821e-16 -> xyz=0.0680211 -0.0776141 -0.0305 rpy=-1.5708 -1.26838 -1.05043e-15; parent still_chassis_assm__configuration_screwless -> still_chassis_assm__configuration_default
- joint rear_left_wheel_speed: child wheel_assm__configuration_screwless_3 -> wheel_assm__configuration_default_3; origin xyz=-0.0804789 0.0783859 -0.0305 rpy=-1.5708 1.53772 -2.56896e-15 -> xyz=-0.0804789 0.0783859 -0.0305 rpy=-1.5708 1.14106 -8.02116e-16; parent still_chassis_assm__configuration_screwless -> still_chassis_assm__configuration_default
- joint rear_right_wheel_speed: child wheel_assm__configuration_screwless_4 -> wheel_assm__configuration_default_4; origin xyz=-0.0804789 -0.0776141 -0.0305 rpy=-1.5708 -1.53772 -1.71073e-14 -> xyz=-0.0804789 -0.0776141 -0.0305 rpy=1.5708 1.46397 -3.14159; parent still_chassis_assm__configuration_screwless -> still_chassis_assm__configuration_default

Commit message: add script to cleanup names and remove configurations

File: src/ballbot_description/onshape/ballbot/robot.urdf (robot description, URDF)
Before this commit: robot ballbot, 6 links, 5 joints
Links:
- removed link still_chassis_assm__configuration_default
- removed link wheel_assm__configuration_default
- removed link wheel_assm__configuration_default_2
- removed link wheel_assm__configuration_default_3
- removed link wheel_assm__configuration_default_4
- added link still_chassis_assm, mass 1.12003; collision box size=0.006 0.014 0.005; collision box size=0.006 0.014 0.005
- added link wheel_assm, mass 0.0544576; collision cylinder length=0.006 radius=0.0069282; collision cylinder length=0.006 radius=0.0069282
- added link wheel_assm_2, mass 0.0544576; collision cylinder length=0.006 radius=0.0069282; collision cylinder length=0.006 radius=0.0069282
- added link wheel_assm_3, mass 0.0544576; collision cylinder length=0.006 radius=0.0069282; collision cylinder length=0.006 radius=0.0069282
- added link wheel_assm_4, mass 0.0544576; collision cylinder length=0.006 radius=0.0069282; collision cylinder length=0.006 radius=0.0069282
Joints:
- removed joint base_link_to_still_chassis_assm__configuration_default
- added joint base_link_to_still_chassis_assm: type fixed, parent base_link, child still_chassis_assm, origin xyz=0 0 0 rpy=0 -0 0, axis 0 0 1, limit effort=10 velocity=10
- joint front_left_wheel_speed: child wheel_assm__configuration_default -> wheel_assm; parent still_chassis_assm__configuration_default -> still_chassis_assm
- joint front_right_wheel_speed: child wheel_assm__configuration_default_2 -> wheel_assm_2; parent still_chassis_assm__configuration_default -> still_chassis_assm
- joint rear_left_wheel_speed: child wheel_assm__configuration_default_3 -> wheel_assm_3; origin xyz=-0.0804789 0.0783859 -0.0305 rpy=-1.5708 1.14106 -8.02116e-16 -> xyz=-0.0804789 0.0783859 -0.0305 rpy=-1.5708 -0.366073 -6.32652e-16; parent still_chassis_assm__configuration_default -> still_chassis_assm
- joint rear_right_wheel_speed: child wheel_assm__configuration_default_4 -> wheel_assm_4; parent still_chassis_assm__configuration_default -> still_chassis_assm

Commit message: fix issue with renaming - only rename links in urdf, not .stl, .part, or .scad

File: src/ballbot_description/onshape/ballbot/robot.urdf (robot description, URDF)
Before this commit: robot ballbot, 6 links, 5 joints
Links:
- link still_chassis_assm: geometry collision box size=0.006 0.014 0.005; collision box size=0.006 0.014 0.005
- link wheel_assm: geometry collision cylinder length=0.006 radius=0.0069282; collision cylinder length=0.006 radius=0.0069282
- link wheel_assm_2: geometry collision cylinder length=0.006 radius=0.0069282; collision cylinder length=0.006 radius=0.0069282
- link wheel_assm_3: geometry collision cylinder length=0.006 radius=0.0069282; collision cylinder length=0.006 radius=0.0069282
- link wheel_assm_4: geometry collision cylinder length=0.006 radius=0.0069282; collision cylinder length=0.006 radius=0.0069282
