Commit message: individual links but they float in bullet right now

File: src/ballbot_description/onshape/ballbot_generated/robot.urdf (robot description, URDF)
Before this commit: robot ballbot_generated, 6 links, 5 joints
Links:
- removed link still_chassis_assm__configuration_default
- removed link wheel_assm__configuration_default
- removed link wheel_assm__configuration_default_2
- removed link wheel_assm__configuration_default_3
- removed link wheel_assm__configuration_default_4
- added link still_chassis_assm, mass 1e-09
- added link still_chassis_assm_chassis_plate, mass 0.143; collision box size=0.242 0.140696 0.002; visual mesh filename=package://assets/chassis_plate__configuration_default.stl
- added link still_chassis_assm_chassis_plate_2, mass 0.143; collision box size=0.242 0.140696 0.002; visual mesh filename=package://assets/chassis_plate__configuration_default.stl
- added link still_chassis_assm_motor_bracket_md520, mass 0.033; collision box size=0.04 0.0035 0.002; collision box size=0.04 0.0035 0.002
- added link still_chassis_assm_motor_bracket_md520_2, mass 0.033; collision box size=0.04 0.0035 0.002; collision box size=0.04 0.0035 0.002
- added link still_chassis_assm_motor_bracket_md520_3, mass 0.033; collision box size=0.04 0.0035 0.002; collision box size=0.04 0.0035 0.002
- added link still_chassis_assm_motor_bracket_md520_4, mass 0.033; collision box size=0.04 0.0035 0.002; collision box size=0.04 0.0035 0.002
- added link still_chassis_assm_motor_md520z30_12v, mass 0.15; collision box size=0.006 0.014 0.005; collision cylinder length=0.006 radius=0.006
- added link still_chassis_assm_motor_md520z30_12v_2, mass 0.15; collision box size=0.006 0.014 0.005; collision cylinder length=0.006 radius=0.006
- added link still_chassis_assm_motor_md520z30_12v_3, mass 0.15; collision box size=0.006 0.014 0.005; collision cylinder length=0.006 radius=0.006
- added link still_chassis_assm_motor_md520z30_12v_4, mass 0.15; collision box size=0.006 0.014 0.005; collision cylinder length=0.006 radius=0.006
- added link still_chassis_assm_spacer_m3_5_60, mass 0.002; collision cylinder length=0.06 radius=0.0025; collision cylinder length=0.06 radius=0.0025
- added link still_chassis_assm_spacer_m3_5_60_2, mass 0.002; collision cylinder length=0.06 radius=0.0025; collision cylinder length=0.06 radius=0.0025
- added link still_chassis_assm_spacer_m3_5_60_3, mass 0.002; collision cylinder length=0.06 radius=0.0025; collision cylinder length=0.06 radius=0.0025
- added link still_chassis_assm_spacer_m3_5_60_4, mass 0.002; collision cylinder length=0.06 radius=0.0025; collision cylinder length=0.06 radius=0.0025
- added link still_chassis_assm_spacer_m3_5_60_5, mass 0.002; collision cylinder length=0.06 radius=0.0025; collision cylinder length=0.06 radius=0.0025
- added link still_chassis_assm_spacer_m3_5_60_6, mass 0.002; collision cylinder length=0.06 radius=0.0025; collision cylinder length=0.06 radius=0.0025
- added link wheel_assm, mass 1e-09
- added link wheel_assm_2, mass 1e-09
- added link wheel_assm_2_hex_coupler_6mm_2, mass 0.013; collision cylinder length=0.006 radius=0.0069282; collision cylinder length=0.006 radius=0.0069282
- added link wheel_assm_2_wheel_2, mass 0.0365; collision cylinder length=0.0265 radius=0.033995; collision cylinder length=0.0265 radius=0.033995
- added link wheel_assm_3, mass 1e-09
- added link wheel_assm_3_hex_coupler_6mm_3, mass 0.013; collision cylinder length=0.006 radius=0.0069282; collision cylinder length=0.006 radius=0.0069282
- added link wheel_assm_3_wheel_3, mass 0.0365; collision cylinder length=0.0265 radius=0.033995; collision cylinder length=0.0265 radius=0.033995
- added link wheel_assm_4, mass 1e-09
- added link wheel_assm_4_hex_coupler_6mm_4, mass 0.013; collision cylinder length=0.006 radius=0.0069282; collision cylinder length=0.006 radius=0.0069282
- added link wheel_assm_4_wheel_4, mass 0.0365; collision cylinder length=0.0265 radius=0.033995; collision cylinder length=0.0265 radius=0.033995
- added link wheel_assm_hex_coupler_6mm, mass 0.013; collision cylinder length=0.006 radius=0.0069282; collision cylinder length=0.006 radius=0.0069282
- added link wheel_assm_wheel, mass 0.0365; collision cylinder length=0.0265 radius=0.033995; collision cylinder length=0.0265 radius=0.033995
Joints:
- removed joint base_link_to_still_chassis_assm__configuration_default
- added joint base_link_to_still_chassis_assm: type fixed, parent base_link, child still_chassis_assm, origin xyz=0 0 0 rpy=0 -0 0, axis 0 0 1, limit effort=10 velocity=10
- added joint still_chassis_assm_chassis_plate_2_fixed: type fixed, parent still_chassis_assm, child still_chassis_assm_chassis_plate_2, origin xyz=-8.50526e-17 -1.0366e-16 0.062 rpy=-5.55112e-17 -6.12323e-17 9.71445e-17, axis 0 0 1, limit effort=10 velocity=10
- added joint still_chassis_assm_chassis_plate_fixed: type fixed, parent still_chassis_assm, child still_chassis_assm_chassis_plate, origin xyz=-5.9848e-17 -8.32667e-17 -4.99115e-18 rpy=-1.26218e-29 -6.12323e-17 9.71445e-17, axis 0 0 1, limit effort=10 velocity=10
- added joint still_chassis_assm_motor_bracket_md520_2_fixed: type fixed, parent still_chassis_assm, child still_chassis_assm_motor_bracket_md520_2, origin xyz=-0.0804789 0.0391359 -0.004 rpy=-1.5708 2.87934e-29 -6.38378e-16, axis 0 0 1, limit effort=10 velocity=10
- added joint still_chassis_assm_motor_bracket_md520_3_fixed: type fixed, parent still_chassis_assm, child still_chassis_assm_motor_bracket_md520_3, origin xyz=-0.0804789 -0.0383641 -0.004 rpy=-1.5708 -1.23753e-29 -3.14159, axis 0 0 1, limit effort=10 velocity=10
- added joint still_chassis_assm_motor_bracket_md520_4_fixed: type fixed, parent still_chassis_assm, child still_chassis_assm_motor_bracket_md520_4, origin xyz=0.0680211 0.0391359 -0.004 rpy=-1.5708 -1.24739e-29 9.71445e-17, axis 0 0 1, limit effort=10 velocity=10
- added joint still_chassis_assm_motor_bracket_md520_fixed: type fixed, parent still_chassis_assm, child still_chassis_assm_motor_bracket_md520, origin xyz=0.0680211 -0.0383641 -0.004 rpy=-1.5708 -2.80046e-29 -3.14159, axis 0 0 1, limit effort=10 velocity=10
- added joint still_chassis_assm_motor_md520z30_12v_2_fixed: type fixed, parent still_chassis_assm, child still_chassis_assm_motor_md520z30_12v_2, origin xyz=-0.0804789 0.0358859 -0.0235 rpy=1.17568e-16 2.64761e-29 -6.55914e-16, axis 0 0 1, limit effort=10 velocity=10
- added joint still_chassis_assm_motor_md520z30_12v_3_fixed: type fixed, parent still_chassis_assm, child still_chassis_assm_motor_md520z30_12v_3, origin xyz=-0.0804789 -0.0351141 -0.0235 rpy=2.84102e-16 -1.46925e-29 -3.14159, axis 0 0 1, limit effort=10 velocity=10
- added joint still_chassis_assm_motor_md520z30_12v_4_fixed: type fixed, parent still_chassis_assm, child still_chassis_assm_motor_md520z30_12v_4, origin xyz=0.0680211 0.0358859 -0.0235 rpy=1.86957e-16 -1.4446e-29 7.96089e-17, axis 0 0 1, limit effort=10 velocity=10
- added joint still_chassis_assm_motor_md520z30_12v_fixed: type fixed, parent still_chassis_assm, child still_chassis_assm_motor_md520z30_12v, origin xyz=0.0680211 -0.0351141 -0.0235 rpy=-1.59987e-16 -3.03218e-29 -3.14159, axis 0 0 1, limit effort=10 velocity=10
- added joint still_chassis_assm_spacer_m3_5_60_2_fixed: type fixed, parent still_chassis_assm, child still_chassis_assm_spacer_m3_5_60_2, origin xyz=-0.00347892 0.0633859 -1.26635e-16 rpy=1.5708 3.22537e-15 8.39606e-16, axis 0 0 1, limit effort=10 velocity=10
- added joint still_chassis_assm_spacer_m3_5_60_3_fixed: type fixed, parent still_chassis_assm, child still_chassis_assm_spacer_m3_5_60_3, origin xyz=0.0830211 0.0503859 9.2427e-20 rpy=1.5708 1.22116e-27 -1.5708, axis 0 0 1, limit effort=10 velocity=10
- added joint still_chassis_assm_spacer_m3_5_60_4_fixed: type fixed, parent still_chassis_assm, child still_chassis_assm_spacer_m3_5_60_4, origin xyz=-0.110479 -0.0576141 3.87034e-19 rpy=1.5708 -1.26218e-29 9.71445e-17, axis 0 0 1, limit effort=10 velocity=10
- added joint still_chassis_assm_spacer_m3_5_60_5_fixed: type fixed, parent still_chassis_assm, child still_chassis_assm_spacer_m3_5_60_5, origin xyz=0.0830211 -0.0496141 9.2427e-20 rpy=1.5708 -1.26218e-29 9.71445e-17, axis 0 0 1, limit effort=10 velocity=10
- added joint still_chassis_assm_spacer_m3_5_60_6_fixed: type fixed, parent still_chassis_assm, child still_chassis_assm_spacer_m3_5_60_6, origin xyz=-0.00347892 -0.0626141 7.88861e-31 rpy=1.5708 -1.80411e-16 -1.5708, axis 0 0 1, limit effort=10 velocity=10
- added joint still_chassis_assm_spacer_m3_5_60_fixed: type fixed, parent still_chassis_assm, child still_chassis_assm_spacer_m3_5_60, origin xyz=-0.110479 0.0583859 3.87034e-19 rpy=1.5708 -1.26218e-29 9.71445e-17, axis 0 0 1, limit effort=10 velocity=10
- added joint wheel_assm_2_hex_coupler_6mm_2_fixed: type fixed, parent wheel_assm_2, child wheel_assm_2_hex_coupler_6mm_2, origin xyz=-1.73472e-18 0 -0.0006 rpy=-1.5708 1.61561e-27 8.31828e-18, axis 0 0 1, limit effort=10 velocity=10
- added joint wheel_assm_2_wheel_2_fixed: type fixed, parent wheel_assm_2, child wheel_assm_2_wheel_2, origin xyz=-4.68375e-17 6.93889e-17 -0.00675 rpy=1.5708 -6.12323e-17 8.31828e-18, axis 0 0 1, limit effort=10 velocity=10
- added joint wheel_assm_3_hex_coupler_6mm_3_fixed: type fixed, parent wheel_assm_3, child wheel_assm_3_hex_coupler_6mm_3, origin xyz=0 3.41524e-18 0.0006 rpy=1.5708 -1.61558e-27 -1.9894e-17, axis 0 0 1, limit effort=10 velocity=10
- added joint wheel_assm_3_wheel_3_fixed: type fixed, parent wheel_assm_3, child wheel_assm_3_wheel_3, origin xyz=1.38778e-17 -3.54534e-17 0.00675 rpy=-1.5708 6.12323e-17 -1.9894e-17, axis 0 0 1, limit effort=10 velocity=10
- added joint wheel_assm_4_hex_coupler_6mm_4_fixed: type fixed, parent wheel_assm_4, child wheel_assm_4_hex_coupler_6mm_4, origin xyz=1.38778e-17 0 -0.0006 rpy=-1.5708 1.61565e-27 1.71228e-17, axis 0 0 1, limit effort=10 velocity=10
- added joint wheel_assm_4_wheel_4_fixed: type fixed, parent wheel_assm_4, child wheel_assm_4_wheel_4, origin xyz=0 2.77556e-17 -0.00675 rpy=1.5708 -6.12323e-17 1.71228e-17, axis 0 0 1, limit effort=10 velocity=10
- added joint wheel_assm_hex_coupler_6mm_fixed: type fixed, parent wheel_assm, child wheel_assm_hex_coupler_6mm, origin xyz=1.38778e-17 -6.93889e-18 0.0006 rpy=1.5708 3.78098e-15 -1.7953, axis 0 0 1, limit effort=10 velocity=10
- added joint wheel_assm_wheel_fixed: type fixed, parent wheel_assm, child wheel_assm_wheel, origin xyz=4.16334e-17 2.08167e-17 0.00675 rpy=-1.5708 3.84221e-15 -1.7953, axis 0 0 1, limit effort=10 velocity=10
- joint front_left_wheel_speed: child wheel_assm__configuration_default -> wheel_assm; parent still_chassis_assm__configuration_default -> still_chassis_assm
- joint front_right_wheel_speed: child wheel_assm__configuration_default_2 -> wheel_assm_2; parent still_chassis_assm__configuration_default -> still_chassis_assm
- joint rear_left_wheel_speed: child wheel_assm__configuration_default_3 -> wheel_assm_3; parent still_chassis_assm__configuration_default -> still_chassis_assm
- joint rear_right_wheel_speed: child wheel_assm__configuration_default_4 -> wheel_assm_4; parent still_chassis_assm__configuration_default -> still_chassis_assm

File: src/ballbot_description/urdf/ballbot.urdf (robot description, URDF)
Before this commit: robot ballbot_generated, 6 links, 5 joints
Links:
- removed link still_chassis_assm__configuration_default
- removed link wheel_assm__configuration_default
- removed link wheel_assm__configuration_default_2
- removed link wheel_assm__configuration_default_3
- removed link wheel_assm__configuration_default_4
- added link still_chassis_assm, mass 1e-09
- added link still_chassis_assm_chassis_plate, mass 0.143; collision box size=0.242 0.140696 0.002; visual mesh filename=package://ballbot_description/meshes/chassis_plate__configu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
- added link still_chassis_assm_chassis_plate_2, mass 0.143; collision box size=0.242 0.140696 0.002; visual mesh filename=package://ballbot_description/meshes/chassis_plate__configu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
- added link still_chassis_assm_motor_bracket_md520, mass 0.033; collision box size=0.04 0.0035 0.002; collision box size=0.04 0.0035 0.002
- added link still_chassis_assm_motor_bracket_md520_2, mass 0.033; collision box size=0.04 0.0035 0.002; collision box size=0.04 0.0035 0.002
- added link still_chassis_assm_motor_bracket_md520_3, mass 0.033; collision box size=0.04 0.0035 0.002; collision box size=0.04 0.0035 0.002
- added link still_chassis_assm_motor_bracket_md520_4, mass 0.033; collision box size=0.04 0.0035 0.002; collision box size=0.04 0.0035 0.002
- added link still_chassis_assm_motor_md520z30_12v, mass 0.15; collision box size=0.006 0.014 0.005; collision cylinder length=0.006 radius=0.006
- added link still_chassis_assm_motor_md520z30_12v_2, mass 0.15; collision box size=0.006 0.014 0.005; collision cylinder length=0.006 radius=0.006
- added link still_chassis_assm_motor_md520z30_12v_3, mass 0.15; collision box size=0.006 0.014 0.005; collision cylinder length=0.006 radius=0.006
- added link still_chassis_assm_motor_md520z30_12v_4, mass 0.15; collision box size=0.006 0.014 0.005; collision cylinder length=0.006 radius=0.006
- added link still_chassis_assm_spacer_m3_5_60, mass 0.002; collision cylinder length=0.06 radius=0.0025; collision cylinder length=0.06 radius=0.0025
- added link still_chassis_assm_spacer_m3_5_60_2, mass 0.002; collision cylinder length=0.06 radius=0.0025; collision cylinder length=0.06 radius=0.0025
- added link still_chassis_assm_spacer_m3_5_60_3, mass 0.002; collision cylinder length=0.06 radius=0.0025; collision cylinder length=0.06 radius=0.0025
- added link still_chassis_assm_spacer_m3_5_60_4, mass 0.002; collision cylinder length=0.06 radius=0.0025; collision cylinder length=0.06 radius=0.0025
- added link still_chassis_assm_spacer_m3_5_60_5, mass 0.002; collision cylinder length=0.06 radius=0.0025; collision cylinder length=0.06 radius=0.0025
- added link still_chassis_assm_spacer_m3_5_60_6, mass 0.002; collision cylinder length=0.06 radius=0.0025; collision cylinder length=0.06 radius=0.0025
- added link wheel_assm, mass 1e-09
- added link wheel_assm_2, mass 1e-09
- added link wheel_assm_2_hex_coupler_6mm_2, mass 0.013; collision cylinder length=0.006 radius=0.0069282; collision cylinder length=0.006 radius=0.0069282
- added link wheel_assm_2_wheel_2, mass 0.0365; collision cylinder length=0.0265 radius=0.033995; collision cylinder length=0.0265 radius=0.033995
- added link wheel_assm_3, mass 1e-09
- added link wheel_assm_3_hex_coupler_6mm_3, mass 0.013; collision cylinder length=0.006 radius=0.0069282; collision cylinder length=0.006 radius=0.0069282
- added link wheel_assm_3_wheel_3, mass 0.0365; collision cylinder length=0.0265 radius=0.033995; collision cylinder length=0.0265 radius=0.033995
- added link wheel_assm_4, mass 1e-09
- added link wheel_assm_4_hex_coupler_6mm_4, mass 0.013; collision cylinder length=0.006 radius=0.0069282; collision cylinder length=0.006 radius=0.0069282
- added link wheel_assm_4_wheel_4, mass 0.0365; collision cylinder length=0.0265 radius=0.033995; collision cylinder length=0.0265 radius=0.033995
- added link wheel_assm_hex_coupler_6mm, mass 0.013; collision cylinder length=0.006 radius=0.0069282; collision cylinder length=0.006 radius=0.0069282
- added link wheel_assm_wheel, mass 0.0365; collision cylinder length=0.0265 radius=0.033995; collision cylinder length=0.0265 radius=0.033995
Joints:
- removed joint base_link_to_still_chassis_assm__configuration_default
- added joint base_link_to_still_chassis_assm: type fixed, parent base_link, child still_chassis_assm, origin xyz=0 0 0 rpy=0 -0 0, axis 0 0 1, limit effort=10 velocity=10
- added joint still_chassis_assm_chassis_plate_2_fixed: type fixed, parent still_chassis_assm, child still_chassis_assm_chassis_plate_2, origin xyz=-8.50526e-17 -1.0366e-16 0.062 rpy=-5.55112e-17 -6.12323e-17 9.71445e-17, axis 0 0 1, limit effort=10 velocity=10
- added joint still_chassis_assm_chassis_plate_fixed: type fixed, parent still_chassis_assm, child still_chassis_assm_chassis_plate, origin xyz=-5.9848e-17 -8.32667e-17 -4.99115e-18 rpy=-1.26218e-29 -6.12323e-17 9.71445e-17, axis 0 0 1, limit effort=10 velocity=10
- added joint still_chassis_assm_motor_bracket_md520_2_fixed: type fixed, parent still_chassis_assm, child still_chassis_assm_motor_bracket_md520_2, origin xyz=-0.0804789 0.0391359 -0.004 rpy=-1.5708 2.87934e-29 -6.38378e-16, axis 0 0 1, limit effort=10 velocity=10
- added joint still_chassis_assm_motor_bracket_md520_3_fixed: type fixed, parent still_chassis_assm, child still_chassis_assm_motor_bracket_md520_3, origin xyz=-0.0804789 -0.0383641 -0.004 rpy=-1.5708 -1.23753e-29 -3.14159, axis 0 0 1, limit effort=10 velocity=10
- added joint still_chassis_assm_motor_bracket_md520_4_fixed: type fixed, parent still_chassis_assm, child still_chassis_assm_motor_bracket_md520_4, origin xyz=0.0680211 0.0391359 -0.004 rpy=-1.5708 -1.24739e-29 9.71445e-17, axis 0 0 1, limit effort=10 velocity=10
- added joint still_chassis_assm_motor_bracket_md520_fixed: type fixed, parent still_chassis_assm, child still_chassis_assm_motor_bracket_md520, origin xyz=0.0680211 -0.0383641 -0.004 rpy=-1.5708 -2.80046e-29 -3.14159, axis 0 0 1, limit effort=10 velocity=10
- added joint still_chassis_assm_motor_md520z30_12v_2_fixed: type fixed, parent still_chassis_assm, child still_chassis_assm_motor_md520z30_12v_2, origin xyz=-0.0804789 0.0358859 -0.0235 rpy=1.17568e-16 2.64761e-29 -6.55914e-16, axis 0 0 1, limit effort=10 velocity=10
- added joint still_chassis_assm_motor_md520z30_12v_3_fixed: type fixed, parent still_chassis_assm, child still_chassis_assm_motor_md520z30_12v_3, origin xyz=-0.0804789 -0.0351141 -0.0235 rpy=2.84102e-16 -1.46925e-29 -3.14159, axis 0 0 1, limit effort=10 velocity=10
- added joint still_chassis_assm_motor_md520z30_12v_4_fixed: type fixed, parent still_chassis_assm, child still_chassis_assm_motor_md520z30_12v_4, origin xyz=0.0680211 0.0358859 -0.0235 rpy=1.86957e-16 -1.4446e-29 7.96089e-17, axis 0 0 1, limit effort=10 velocity=10
- added joint still_chassis_assm_motor_md520z30_12v_fixed: type fixed, parent still_chassis_assm, child still_chassis_assm_motor_md520z30_12v, origin xyz=0.0680211 -0.0351141 -0.0235 rpy=-1.59987e-16 -3.03218e-29 -3.14159, axis 0 0 1, limit effort=10 velocity=10
- added joint still_chassis_assm_spacer_m3_5_60_2_fixed: type fixed, parent still_chassis_assm, child still_chassis_assm_spacer_m3_5_60_2, origin xyz=-0.00347892 0.0633859 -1.26635e-16 rpy=1.5708 3.22537e-15 8.39606e-16, axis 0 0 1, limit effort=10 velocity=10
- added joint still_chassis_assm_spacer_m3_5_60_3_fixed: type fixed, parent still_chassis_assm, child still_chassis_assm_spacer_m3_5_60_3, origin xyz=0.0830211 0.0503859 9.2427e-20 rpy=1.5708 1.22116e-27 -1.5708, axis 0 0 1, limit effort=10 velocity=10
- added joint still_chassis_assm_spacer_m3_5_60_4_fixed: type fixed, parent still_chassis_assm, child still_chassis_assm_spacer_m3_5_60_4, origin xyz=-0.110479 -0.0576141 3.87034e-19 rpy=1.5708 -1.26218e-29 9.71445e-17, axis 0 0 1, limit effort=10 velocity=10
- added joint still_chassis_assm_spacer_m3_5_60_5_fixed: type fixed, parent still_chassis_assm, child still_chassis_assm_spacer_m3_5_60_5, origin xyz=0.0830211 -0.0496141 9.2427e-20 rpy=1.5708 -1.26218e-29 9.71445e-17, axis 0 0 1, limit effort=10 velocity=10
- added joint still_chassis_assm_spacer_m3_5_60_6_fixed: type fixed, parent still_chassis_assm, child still_chassis_assm_spacer_m3_5_60_6, origin xyz=-0.00347892 -0.0626141 7.88861e-31 rpy=1.5708 -1.80411e-16 -1.5708, axis 0 0 1, limit effort=10 velocity=10
- added joint still_chassis_assm_spacer_m3_5_60_fixed: type fixed, parent still_chassis_assm, child still_chassis_assm_spacer_m3_5_60, origin xyz=-0.110479 0.0583859 3.87034e-19 rpy=1.5708 -1.26218e-29 9.71445e-17, axis 0 0 1, limit effort=10 velocity=10
- added joint wheel_assm_2_hex_coupler_6mm_2_fixed: type fixed, parent wheel_assm_2, child wheel_assm_2_hex_coupler_6mm_2, origin xyz=-1.73472e-18 0 -0.0006 rpy=-1.5708 1.61561e-27 8.31828e-18, axis 0 0 1, limit effort=10 velocity=10
- added joint wheel_assm_2_wheel_2_fixed: type fixed, parent wheel_assm_2, child wheel_assm_2_wheel_2, origin xyz=-4.68375e-17 6.93889e-17 -0.00675 rpy=1.5708 -6.12323e-17 8.31828e-18, axis 0 0 1, limit effort=10 velocity=10
- added joint wheel_assm_3_hex_coupler_6mm_3_fixed: type fixed, parent wheel_assm_3, child wheel_assm_3_hex_coupler_6mm_3, origin xyz=0 3.41524e-18 0.0006 rpy=1.5708 -1.61558e-27 -1.9894e-17, axis 0 0 1, limit effort=10 velocity=10
- added joint wheel_assm_3_wheel_3_fixed: type fixed, parent wheel_assm_3, child wheel_assm_3_wheel_3, origin xyz=1.38778e-17 -3.54534e-17 0.00675 rpy=-1.5708 6.12323e-17 -1.9894e-17, axis 0 0 1, limit effort=10 velocity=10
- added joint wheel_assm_4_hex_coupler_6mm_4_fixed: type fixed, parent wheel_assm_4, child wheel_assm_4_hex_coupler_6mm_4, origin xyz=1.38778e-17 0 -0.0006 rpy=-1.5708 1.61565e-27 1.71228e-17, axis 0 0 1, limit effort=10 velocity=10
- added joint wheel_assm_4_wheel_4_fixed: type fixed, parent wheel_assm_4, child wheel_assm_4_wheel_4, origin xyz=0 2.77556e-17 -0.00675 rpy=1.5708 -6.12323e-17 1.71228e-17, axis 0 0 1, limit effort=10 velocity=10
- added joint wheel_assm_hex_coupler_6mm_fixed: type fixed, parent wheel_assm, child wheel_assm_hex_coupler_6mm, origin xyz=1.38778e-17 -6.93889e-18 0.0006 rpy=1.5708 3.78098e-15 -1.7953, axis 0 0 1, limit effort=10 velocity=10
- added joint wheel_assm_wheel_fixed: type fixed, parent wheel_assm, child wheel_assm_wheel, origin xyz=4.16334e-17 2.08167e-17 0.00675 rpy=-1.5708 3.84221e-15 -1.7953, axis 0 0 1, limit effort=10 velocity=10
- joint front_left_wheel_speed: child wheel_assm__configuration_default -> wheel_assm; parent still_chassis_assm__configuration_default -> still_chassis_assm
- joint front_right_wheel_speed: child wheel_assm__configuration_default_2 -> wheel_assm_2; parent still_chassis_assm__configuration_default -> still_chassis_assm
- joint rear_left_wheel_speed: child wheel_assm__configuration_default_3 -> wheel_assm_3; parent still_chassis_assm__configuration_default -> still_chassis_assm
- joint rear_right_wheel_speed: child wheel_assm__configuration_default_4 -> wheel_assm_4; parent still_chassis_assm__configuration_default -> still_chassis_assm
