Commit message: add rplidar - stls not merged right

File: src/ballbot_description/onshape/ballbot_generated/robot.urdf (robot description, URDF)
Before this commit: robot ballbot_generated, 30 links, 29 joints
Links:
- added link still_chassis_assm_base_ipt, mass 0.0178296; visual mesh filename=package://assets/base_ipt.stl
- added link still_chassis_assm_bn_3318_3664352_hex_stand_off_m2_5x16, mass 0.00294966; visual mesh filename=package://assets/bn_3318_3664352_hex_stand_off_m2_5x16.stl
- added link still_chassis_assm_bn_3318_3664352_hex_stand_off_m2_5x16_10, mass 0.00294966; visual mesh filename=package://assets/bn_3318_3664352_hex_stand_off_m2_5x16.stl
- added link still_chassis_assm_bn_3318_3664352_hex_stand_off_m2_5x16_11, mass 0.00294966; visual mesh filename=package://assets/bn_3318_3664352_hex_stand_off_m2_5x16.stl
- added link still_chassis_assm_bn_3318_3664352_hex_stand_off_m2_5x16_12, mass 0.00294966; visual mesh filename=package://assets/bn_3318_3664352_hex_stand_off_m2_5x16.stl
- added link still_chassis_assm_bn_3318_3664352_hex_stand_off_m2_5x16_2, mass 0.00294966; visual mesh filename=package://assets/bn_3318_3664352_hex_stand_off_m2_5x16.stl
- added link still_chassis_assm_bn_3318_3664352_hex_stand_off_m2_5x16_3, mass 0.00294966; visual mesh filename=package://assets/bn_3318_3664352_hex_stand_off_m2_5x16.stl
- added link still_chassis_assm_bn_3318_3664352_hex_stand_off_m2_5x16_4, mass 0.00294966; visual mesh filename=package://assets/bn_3318_3664352_hex_stand_off_m2_5x16.stl
- added link still_chassis_assm_bn_3318_3664352_hex_stand_off_m2_5x16_5, mass 0.00294966; visual mesh filename=package://assets/bn_3318_3664352_hex_stand_off_m2_5x16.stl
- added link still_chassis_assm_bn_3318_3664352_hex_stand_off_m2_5x16_6, mass 0.00294966; visual mesh filename=package://assets/bn_3318_3664352_hex_stand_off_m2_5x16.stl
- added link still_chassis_assm_bn_3318_3664352_hex_stand_off_m2_5x16_7, mass 0.00294966; visual mesh filename=package://assets/bn_3318_3664352_hex_stand_off_m2_5x16.stl
- added link still_chassis_assm_bn_3318_3664352_hex_stand_off_m2_5x16_8, mass 0.00294966; visual mesh filename=package://assets/bn_3318_3664352_hex_stand_off_m2_5x16.stl
- added link still_chassis_assm_bn_3318_3664352_hex_stand_off_m2_5x16_9, mass 0.00294966; visual mesh filename=package://assets/bn_3318_3664352_hex_stand_off_m2_5x16.stl
- added link still_chassis_assm_connector_1_25_3pin_ipt, mass 5.87188e-05; visual mesh filename=package://assets/connector_1_25_3pin_ipt.stl
- added link still_chassis_assm_connector_1_25_4pin_ipt, mass 6.37994e-05; visual mesh filename=package://assets/connector_1_25_4pin_ipt.stl
- added link still_chassis_assm_detector_ipt, mass 0.00982014; visual mesh filename=package://assets/detector_ipt.stl
- added link still_chassis_assm_detector_mount_ipt, mass 0.00130069; visual mesh filename=package://assets/detector_mount_ipt.stl
- added link still_chassis_assm_head_base_ipt, mass 0.0122368; visual mesh filename=package://assets/head_base_ipt.stl
- added link still_chassis_assm_head_ipt, mass 0.00711679; visual mesh filename=package://assets/head_ipt.stl
- added link still_chassis_assm_laser_ipt, mass 0.00497222; visual mesh filename=package://assets/laser_ipt.stl
- added link still_chassis_assm_laser_mount_ipt, mass 0.000744536; visual mesh filename=package://assets/laser_mount_ipt.stl
- added link still_chassis_assm_motherboard_ipt, mass 0.00295286; visual mesh filename=package://assets/motherboard_ipt.stl
- added link still_chassis_assm_motor_board_ipt, mass 0.00127935; visual mesh filename=package://assets/motor_board_ipt.stl
- added link still_chassis_assm_motor_ipt, mass 0.131981; visual mesh filename=package://assets/motor_ipt.stl
- added link still_chassis_assm_rubber_ipt, mass 0.00083994; visual mesh filename=package://assets/rubber_ipt.stl
- added link still_chassis_assm_wheel_ipt, mass 0.000740487; visual mesh filename=package://assets/wheel_ipt.stl
- added link still_chassis_assm_woodscrews_gb_type136_m2x6_n_ipt, mass 7.63832e-05
- added link still_chassis_assm_woodscrews_gb_type136_m2x6_n_ipt_2, mass 7.63832e-05
- added link still_chassis_assm_woodscrews_gb_type136_m2x6_n_ipt_3, mass 7.63832e-05
- added link still_chassis_assm_woodscrews_gb_type136_m2x6_n_ipt_4, mass 7.63832e-05
- added link still_chassis_assm_woodscrews_gb_type136_m2x6_n_ipt_5, mass 7.63832e-05
Joints:
- added joint still_chassis_assm_base_ipt_fixed: type fixed, parent still_chassis_assm, child still_chassis_assm_base_ipt, origin xyz=0.0855211 0.000385868 0.114 rpy=7.70228e-28 1.52349e-29 -3.14159, axis 0 0 1, limit effort=10 velocity=10
- added joint still_chassis_assm_bn_3318_3664352_hex_stand_off_m2_5x16_10_fixed: type fixed, parent still_chassis_assm, child still_chassis_assm_bn_3318_3664352_hex_stand_off_m2_5x16_10, origin xyz=0.0435211 0.0203859 0.094 rpy=-2.84495e-16 1.5708 0, axis 0 0 1, limit effort=10 velocity=10
- added joint still_chassis_assm_bn_3318_3664352_hex_stand_off_m2_5x16_11_fixed: type fixed, parent still_chassis_assm, child still_chassis_assm_bn_3318_3664352_hex_stand_off_m2_5x16_11, origin xyz=0.0435211 0.0203859 0.078 rpy=-2.84495e-16 1.5708 0, axis 0 0 1, limit effort=10 velocity=10
- added joint still_chassis_assm_bn_3318_3664352_hex_stand_off_m2_5x16_12_fixed: type fixed, parent still_chassis_assm, child still_chassis_assm_bn_3318_3664352_hex_stand_off_m2_5x16_12, origin xyz=0.0435211 0.0203859 0.11 rpy=-2.84495e-16 1.5708 0, axis 0 0 1, limit effort=10 velocity=10
- added joint still_chassis_assm_bn_3318_3664352_hex_stand_off_m2_5x16_2_fixed: type fixed, parent still_chassis_assm, child still_chassis_assm_bn_3318_3664352_hex_stand_off_m2_5x16_2, origin xyz=0.113521 0.0283859 0.078 rpy=-2.84495e-16 1.5708 0, axis 0 0 1, limit effort=10 velocity=10
- added joint still_chassis_assm_bn_3318_3664352_hex_stand_off_m2_5x16_3_fixed: type fixed, parent still_chassis_assm, child still_chassis_assm_bn_3318_3664352_hex_stand_off_m2_5x16_3, origin xyz=0.113521 0.0283859 0.11 rpy=-2.84495e-16 1.5708 0, axis 0 0 1, limit effort=10 velocity=10
- added joint still_chassis_assm_bn_3318_3664352_hex_stand_off_m2_5x16_4_fixed: type fixed, parent still_chassis_assm, child still_chassis_assm_bn_3318_3664352_hex_stand_off_m2_5x16_4, origin xyz=0.113521 -0.0276141 0.094 rpy=-2.84495e-16 1.5708 0, axis 0 0 1, limit effort=10 velocity=10
- added joint still_chassis_assm_bn_3318_3664352_hex_stand_off_m2_5x16_5_fixed: type fixed, parent still_chassis_assm, child still_chassis_assm_bn_3318_3664352_hex_stand_off_m2_5x16_5, origin xyz=0.113521 -0.0276141 0.078 rpy=-2.84495e-16 1.5708 0, axis 0 0 1, limit effort=10 velocity=10
- added joint still_chassis_assm_bn_3318_3664352_hex_stand_off_m2_5x16_6_fixed: type fixed, parent still_chassis_assm, child still_chassis_assm_bn_3318_3664352_hex_stand_off_m2_5x16_6, origin xyz=0.113521 -0.0276141 0.11 rpy=-2.84495e-16 1.5708 0, axis 0 0 1, limit effort=10 velocity=10
- added joint still_chassis_assm_bn_3318_3664352_hex_stand_off_m2_5x16_7_fixed: type fixed, parent still_chassis_assm, child still_chassis_assm_bn_3318_3664352_hex_stand_off_m2_5x16_7, origin xyz=0.0435211 -0.0196141 0.094 rpy=-2.84495e-16 1.5708 0, axis 0 0 1, limit effort=10 velocity=10
- added joint still_chassis_assm_bn_3318_3664352_hex_stand_off_m2_5x16_8_fixed: type fixed, parent still_chassis_assm, child still_chassis_assm_bn_3318_3664352_hex_stand_off_m2_5x16_8, origin xyz=0.0435211 -0.0196141 0.078 rpy=-2.84495e-16 1.5708 0, axis 0 0 1, limit effort=10 velocity=10
- added joint still_chassis_assm_bn_3318_3664352_hex_stand_off_m2_5x16_9_fixed: type fixed, parent still_chassis_assm, child still_chassis_assm_bn_3318_3664352_hex_stand_off_m2_5x16_9, origin xyz=0.0435211 -0.0196141 0.11 rpy=-2.84495e-16 1.5708 0, axis 0 0 1, limit effort=10 velocity=10
- added joint still_chassis_assm_bn_3318_3664352_hex_stand_off_m2_5x16_fixed: type fixed, parent still_chassis_assm, child still_chassis_assm_bn_3318_3664352_hex_stand_off_m2_5x16, origin xyz=0.113521 0.0283859 0.094 rpy=-2.84495e-16 1.5708 0, axis 0 0 1, limit effort=10 velocity=10
- added joint still_chassis_assm_connector_1_25_3pin_ipt_fixed: type fixed, parent still_chassis_assm, child still_chassis_assm_connector_1_25_3pin_ipt, origin xyz=0.0525211 2.33735e-05 0.0892 rpy=1.5708 -2.44929e-16 1.5708, axis 0 0 1, limit effort=10 velocity=10
- added joint still_chassis_assm_connector_1_25_4pin_ipt_fixed: type fixed, parent still_chassis_assm, child still_chassis_assm_connector_1_25_4pin_ipt, origin xyz=0.0633211 0.000260868 0.10215 rpy=-3.14159 -1.22465e-16 1.5708, axis 0 0 1, limit effort=10 velocity=10
- added joint still_chassis_assm_detector_ipt_fixed: type fixed, parent still_chassis_assm, child still_chassis_assm_detector_ipt, origin xyz=0.0882947 0.0205619 0.129 rpy=3.14159 -1.36674 -1.11796, axis 0 0 1, limit effort=10 velocity=10
- added joint still_chassis_assm_detector_mount_ipt_fixed: type fixed, parent still_chassis_assm, child still_chassis_assm_detector_mount_ipt, origin xyz=0.0853916 0.000243904 0.12 rpy=-2.66271e-13 1.72854e-13 -1.11796, axis 0 0 1, limit effort=10 velocity=10
- added joint still_chassis_assm_head_base_ipt_fixed: type fixed, parent still_chassis_assm, child still_chassis_assm_head_base_ipt, origin xyz=0.0855211 0.000385868 0.117 rpy=-9.16055e-14 -1.4551e-13 -2.69096, axis 0 0 1, limit effort=10 velocity=10
- added joint still_chassis_assm_head_ipt_fixed: type fixed, parent still_chassis_assm, child still_chassis_assm_head_ipt, origin xyz=0.0855211 0.000385868 0.1389 rpy=-3.14159 -9.16055e-14 2.02143, axis 0 0 1, limit effort=10 velocity=10
- added joint still_chassis_assm_laser_ipt_fixed: type fixed, parent still_chassis_assm, child still_chassis_assm_laser_ipt, origin xyz=0.0910946 -0.0247055 0.13 rpy=2.70738e-13 -0.804343 2.15543, axis 0 0 1, limit effort=10 velocity=10
- added joint still_chassis_assm_laser_mount_ipt_fixed: type fixed, parent still_chassis_assm, child still_chassis_assm_laser_mount_ipt, origin xyz=0.0855211 0.000385868 0.121 rpy=-2.81973e-13 1.55655e-13 -1.12579, axis 0 0 1, limit effort=10 velocity=10
- added joint still_chassis_assm_motherboard_ipt_fixed: type fixed, parent still_chassis_assm, child still_chassis_assm_motherboard_ipt, origin xyz=0.0855211 0.000385868 0.104 rpy=7.70228e-28 1.52349e-29 -3.14159, axis 0 0 1, limit effort=10 velocity=10
- added joint still_chassis_assm_motor_board_ipt_fixed: type fixed, parent still_chassis_assm, child still_chassis_assm_motor_board_ipt, origin xyz=0.0400211 0.000385868 0.0909 rpy=-1.98086e-16 -1.26575e-16 2.0044, axis 0 0 1, limit effort=10 velocity=10
- added joint still_chassis_assm_motor_ipt_fixed: type fixed, parent still_chassis_assm, child still_chassis_assm_motor_ipt, origin xyz=0.0400211 0.000385868 0.0945 rpy=-6.12279e-17 -1.84437e-16 1.5708, axis 0 0 1, limit effort=10 velocity=10
- added joint still_chassis_assm_rubber_ipt_fixed: type fixed, parent still_chassis_assm, child still_chassis_assm_rubber_ipt, origin xyz=0.0855211 0.000385868 0.117186 rpy=1.5708 -1.37204e-16 -3.14159, axis 0 0 1, limit effort=10 velocity=10
- added joint still_chassis_assm_wheel_ipt_fixed: type fixed, parent still_chassis_assm, child still_chassis_assm_wheel_ipt, origin xyz=0.0400211 0.000385868 0.115 rpy=1.28639e-16 3.79626e-17 -1.44637, axis 0 0 1, limit effort=10 velocity=10
- added joint still_chassis_assm_woodscrews_gb_type136_m2x6_n_ipt_2_fixed: type fixed, parent still_chassis_assm, child still_chassis_assm_woodscrews_gb_type136_m2x6_n_ipt_2, origin xyz=0.0591707 0.00985469 0.1325 rpy=-1.06785 1.5708 0, axis 0 0 1, limit effort=10 velocity=10
- added joint still_chassis_assm_woodscrews_gb_type136_m2x6_n_ipt_3_fixed: type fixed, parent still_chassis_assm, child still_chassis_assm_woodscrews_gb_type136_m2x6_n_ipt_3, origin xyz=0.076592 -0.0261522 0.1325 rpy=-1.06785 1.5708 0, axis 0 0 1, limit effort=10 velocity=10
- added joint still_chassis_assm_woodscrews_gb_type136_m2x6_n_ipt_4_fixed: type fixed, parent still_chassis_assm, child still_chassis_assm_woodscrews_gb_type136_m2x6_n_ipt_4, origin xyz=0.0400211 0.0113859 0.1163 rpy=3.10866 1.5708 0, axis 0 0 1, limit effort=10 velocity=10
- added joint still_chassis_assm_woodscrews_gb_type136_m2x6_n_ipt_5_fixed: type fixed, parent still_chassis_assm, child still_chassis_assm_woodscrews_gb_type136_m2x6_n_ipt_5, origin xyz=0.0400211 -0.0106141 0.1163 rpy=3.10866 1.5708 0, axis 0 0 1, limit effort=10 velocity=10
- added joint still_chassis_assm_woodscrews_gb_type136_m2x6_n_ipt_fixed: type fixed, parent still_chassis_assm, child still_chassis_assm_woodscrews_gb_type136_m2x6_n_ipt, origin xyz=0.110726 0.0125808 0.1325 rpy=-1.17437 1.5708 0, axis 0 0 1, limit effort=10 velocity=10
