Commit message: merge stls re-enabled

File: src/ballbot_description/onshape/ballbot_generated/robot.urdf (robot description, URDF)
Before this commit: robot ballbot_generated, 62 links, 61 joints
Links:
- removed link rplidar_a1_head_detector_ipt
- removed link rplidar_a1_head_detector_mount_ipt
- removed link rplidar_a1_head_head_ipt
- removed link rplidar_a1_head_laser_ipt
- removed link rplidar_a1_head_laser_mount_ipt
- removed link rplidar_a1_head_woodscrews_gb_type136_m2x6_n_ipt_3
- removed link rplidar_a1_head_woodscrews_gb_type136_m2x6_n_ipt_4
- removed link rplidar_a1_head_woodscrews_gb_type136_m2x6_n_ipt_5
- removed link still_chassis_assm_base_ipt
- removed link still_chassis_assm_bn_3318_3664352_hex_stand_off_m2_5x16
- removed link still_chassis_assm_bn_3318_3664352_hex_stand_off_m2_5x16_10
- removed link still_chassis_assm_bn_3318_3664352_hex_stand_off_m2_5x16_11
- removed link still_chassis_assm_bn_3318_3664352_hex_stand_off_m2_5x16_12
- removed link still_chassis_assm_bn_3318_3664352_hex_stand_off_m2_5x16_2
- removed link still_chassis_assm_bn_3318_3664352_hex_stand_off_m2_5x16_3
- removed link still_chassis_assm_bn_3318_3664352_hex_stand_off_m2_5x16_4
- removed link still_chassis_assm_bn_3318_3664352_hex_stand_off_m2_5x16_5
- removed link still_chassis_assm_bn_3318_3664352_hex_stand_off_m2_5x16_6
- removed link still_chassis_assm_bn_3318_3664352_hex_stand_off_m2_5x16_7
- removed link still_chassis_assm_bn_3318_3664352_hex_stand_off_m2_5x16_8
- removed link still_chassis_assm_bn_3318_3664352_hex_stand_off_m2_5x16_9
- removed link still_chassis_assm_chassis_plate
- removed link still_chassis_assm_chassis_plate_2
- removed link still_chassis_assm_connector_1_25_3pin_ipt
- removed link still_chassis_assm_connector_1_25_4pin_ipt
- removed link still_chassis_assm_head_base_ipt
- removed link still_chassis_assm_motherboard_ipt
- removed link still_chassis_assm_motor_board_ipt
- removed link still_chassis_assm_motor_bracket_md520
- removed link still_chassis_assm_motor_bracket_md520_2
- removed link still_chassis_assm_motor_bracket_md520_3
- removed link still_chassis_assm_motor_bracket_md520_4
- removed link still_chassis_assm_motor_ipt
- removed link still_chassis_assm_motor_md520z30_12v
- removed link still_chassis_assm_motor_md520z30_12v_2
- removed link still_chassis_assm_motor_md520z30_12v_3
- removed link still_chassis_assm_motor_md520z30_12v_4
- removed link still_chassis_assm_rubber_ipt
- removed link still_chassis_assm_spacer_m3_5_60
- removed link still_chassis_assm_spacer_m3_5_60_2
- removed link still_chassis_assm_spacer_m3_5_60_3
- removed link still_chassis_assm_spacer_m3_5_60_4
- removed link still_chassis_assm_spacer_m3_5_60_5
- removed link still_chassis_assm_spacer_m3_5_60_6
- removed link still_chassis_assm_wheel_ipt
- removed link still_chassis_assm_woodscrews_gb_type136_m2x6_n_ipt
- removed link still_chassis_assm_woodscrews_gb_type136_m2x6_n_ipt_2
- removed link wheel_assm_2_hex_coupler_6mm_2
- removed link wheel_assm_2_wheel_2
- removed link wheel_assm_3_hex_coupler_6mm_3
- removed link wheel_assm_3_wheel_3
- removed link wheel_assm_4_hex_coupler_6mm_4
- removed link wheel_assm_4_wheel_4
- removed link wheel_assm_hex_coupler_6mm
- removed link wheel_assm_wheel
- link rplidar_a1_head: mass 1e-09 -> 0.0241835; geometry collision cylinder length=0.02 radius=0.0336123; collision cylinder length=0.02 radius=0.034612
- link still_chassis_assm: mass 1e-09 -> 1.23353; geometry collision box size=0.006 0.014 0.005; collision box size=0.006 0.014 0.005
- link wheel_assm: mass 1e-09 -> 0.0495; geometry collision cylinder length=0.006 radius=0.0069282; collision cylinder length=0.006 radius=0.0069282
- link wheel_assm_2: mass 1e-09 -> 0.0495; geometry collision cylinder length=0.006 radius=0.0069282; collision cylinder length=0.006 radius=0.0069282
- link wheel_assm_3: mass 1e-09 -> 0.0495; geometry collision cylinder length=0.006 radius=0.0069282; collision cylinder length=0.006 radius=0.0069282
- link wheel_assm_4: mass 1e-09 -> 0.0495; geometry collision cylinder length=0.006 radius=0.0069282; collision cylinder length=0.006 radius=0.0069282
Joints:
- removed joint rplidar_a1_head_detector_ipt_fixed
- removed joint rplidar_a1_head_detector_mount_ipt_fixed
- removed joint rplidar_a1_head_head_ipt_fixed
- removed joint rplidar_a1_head_laser_ipt_fixed
- removed joint rplidar_a1_head_laser_mount_ipt_fixed
- removed joint rplidar_a1_head_woodscrews_gb_type136_m2x6_n_ipt_3_fixed
- removed joint rplidar_a1_head_woodscrews_gb_type136_m2x6_n_ipt_4_fixed
- removed joint rplidar_a1_head_woodscrews_gb_type136_m2x6_n_ipt_5_fixed
- removed joint still_chassis_assm_base_ipt_fixed
- removed joint still_chassis_assm_bn_3318_3664352_hex_stand_off_m2_5x16_10_fixed
- removed joint still_chassis_assm_bn_3318_3664352_hex_stand_off_m2_5x16_11_fixed
- removed joint still_chassis_assm_bn_3318_3664352_hex_stand_off_m2_5x16_12_fixed
- removed joint still_chassis_assm_bn_3318_3664352_hex_stand_off_m2_5x16_2_fixed
- removed joint still_chassis_assm_bn_3318_3664352_hex_stand_off_m2_5x16_3_fixed
- removed joint still_chassis_assm_bn_3318_3664352_hex_stand_off_m2_5x16_4_fixed
- removed joint still_chassis_assm_bn_3318_3664352_hex_stand_off_m2_5x16_5_fixed
- removed joint still_chassis_assm_bn_3318_3664352_hex_stand_off_m2_5x16_6_fixed
- removed joint still_chassis_assm_bn_3318_3664352_hex_stand_off_m2_5x16_7_fixed
- removed joint still_chassis_assm_bn_3318_3664352_hex_stand_off_m2_5x16_8_fixed
- removed joint still_chassis_assm_bn_3318_3664352_hex_stand_off_m2_5x16_9_fixed
- removed joint still_chassis_assm_bn_3318_3664352_hex_stand_off_m2_5x16_fixed
- removed joint still_chassis_assm_chassis_plate_2_fixed
- removed joint still_chassis_assm_chassis_plate_fixed
- removed joint still_chassis_assm_connector_1_25_3pin_ipt_fixed
- removed joint still_chassis_assm_connector_1_25_4pin_ipt_fixed
- removed joint still_chassis_assm_head_base_ipt_fixed
- removed joint still_chassis_assm_motherboard_ipt_fixed
- removed joint still_chassis_assm_motor_board_ipt_fixed
- removed joint still_chassis_assm_motor_bracket_md520_2_fixed
- removed joint still_chassis_assm_motor_bracket_md520_3_fixed
- removed joint still_chassis_assm_motor_bracket_md520_4_fixed
- removed joint still_chassis_assm_motor_bracket_md520_fixed
- removed joint still_chassis_assm_motor_ipt_fixed
- removed joint still_chassis_assm_motor_md520z30_12v_2_fixed
- removed joint still_chassis_assm_motor_md520z30_12v_3_fixed
- removed joint still_chassis_assm_motor_md520z30_12v_4_fixed
- removed joint still_chassis_assm_motor_md520z30_12v_fixed
- removed joint still_chassis_assm_rubber_ipt_fixed
- removed joint still_chassis_assm_spacer_m3_5_60_2_fixed
- removed joint still_chassis_assm_spacer_m3_5_60_3_fixed
- removed joint still_chassis_assm_spacer_m3_5_60_4_fixed
- removed joint still_chassis_assm_spacer_m3_5_60_5_fixed
- removed joint still_chassis_assm_spacer_m3_5_60_6_fixed
- removed joint still_chassis_assm_spacer_m3_5_60_fixed
- removed joint still_chassis_assm_wheel_ipt_fixed
- removed joint still_chassis_assm_woodscrews_gb_type136_m2x6_n_ipt_2_fixed
- removed joint still_chassis_assm_woodscrews_gb_type136_m2x6_n_ipt_fixed
- removed joint wheel_assm_2_hex_coupler_6mm_2_fixed
- removed joint wheel_assm_2_wheel_2_fixed
- removed joint wheel_assm_3_hex_coupler_6mm_3_fixed
- removed joint wheel_assm_3_wheel_3_fixed
- removed joint wheel_assm_4_hex_coupler_6mm_4_fixed
- removed joint wheel_assm_4_wheel_4_fixed
- removed joint wheel_assm_hex_coupler_6mm_fixed
- removed joint wheel_assm_wheel_fixed

File: src/ballbot_description/urdf/ballbot.urdf (robot description, URDF)
Before this commit: robot ballbot_generated, 62 links, 61 joints
Links:
- removed link rplidar_a1_head_detector_ipt
- removed link rplidar_a1_head_detector_mount_ipt
- removed link rplidar_a1_head_head_ipt
- removed link rplidar_a1_head_laser_ipt
- removed link rplidar_a1_head_laser_mount_ipt
- removed link rplidar_a1_head_woodscrews_gb_type136_m2x6_n_ipt_3
- removed link rplidar_a1_head_woodscrews_gb_type136_m2x6_n_ipt_4
- removed link rplidar_a1_head_woodscrews_gb_type136_m2x6_n_ipt_5
- removed link still_chassis_assm_base_ipt
- removed link still_chassis_assm_bn_3318_3664352_hex_stand_off_m2_5x16
- removed link still_chassis_assm_bn_3318_3664352_hex_stand_off_m2_5x16_10
- removed link still_chassis_assm_bn_3318_3664352_hex_stand_off_m2_5x16_11
- removed link still_chassis_assm_bn_3318_3664352_hex_stand_off_m2_5x16_12
- removed link still_chassis_assm_bn_3318_3664352_hex_stand_off_m2_5x16_2
- removed link still_chassis_assm_bn_3318_3664352_hex_stand_off_m2_5x16_3
- removed link still_chassis_assm_bn_3318_3664352_hex_stand_off_m2_5x16_4
- removed link still_chassis_assm_bn_3318_3664352_hex_stand_off_m2_5x16_5
- removed link still_chassis_assm_bn_3318_3664352_hex_stand_off_m2_5x16_6
- removed link still_chassis_assm_bn_3318_3664352_hex_stand_off_m2_5x16_7
- removed link still_chassis_assm_bn_3318_3664352_hex_stand_off_m2_5x16_8
- removed link still_chassis_assm_bn_3318_3664352_hex_stand_off_m2_5x16_9
- removed link still_chassis_assm_chassis_plate
- removed link still_chassis_assm_chassis_plate_2
- removed link still_chassis_assm_connector_1_25_3pin_ipt
- removed link still_chassis_assm_connector_1_25_4pin_ipt
- removed link still_chassis_assm_head_base_ipt
- removed link still_chassis_assm_motherboard_ipt
- removed link still_chassis_assm_motor_board_ipt
- removed link still_chassis_assm_motor_bracket_md520
- removed link still_chassis_assm_motor_bracket_md520_2
- removed link still_chassis_assm_motor_bracket_md520_3
- removed link still_chassis_assm_motor_bracket_md520_4
- removed link still_chassis_assm_motor_ipt
- removed link still_chassis_assm_motor_md520z30_12v
- removed link still_chassis_assm_motor_md520z30_12v_2
- removed link still_chassis_assm_motor_md520z30_12v_3
- removed link still_chassis_assm_motor_md520z30_12v_4
- removed link still_chassis_assm_rubber_ipt
- removed link still_chassis_assm_spacer_m3_5_60
- removed link still_chassis_assm_spacer_m3_5_60_2
- removed link still_chassis_assm_spacer_m3_5_60_3
- removed link still_chassis_assm_spacer_m3_5_60_4
- removed link still_chassis_assm_spacer_m3_5_60_5
- removed link still_chassis_assm_spacer_m3_5_60_6
- removed link still_chassis_assm_wheel_ipt
- removed link still_chassis_assm_woodscrews_gb_type136_m2x6_n_ipt
- removed link still_chassis_assm_woodscrews_gb_type136_m2x6_n_ipt_2
- removed link wheel_assm_2_hex_coupler_6mm_2
- removed link wheel_assm_2_wheel_2
- removed link wheel_assm_3_hex_coupler_6mm_3
- removed link wheel_assm_3_wheel_3
- removed link wheel_assm_4_hex_coupler_6mm_4
- removed link wheel_assm_4_wheel_4
- removed link wheel_assm_hex_coupler_6mm
- removed link wheel_assm_wheel
- link rplidar_a1_head: mass 1e-09 -> 0.0241835; geometry collision cylinder length=0.02 radius=0.0336123; collision cylinder length=0.02 radius=0.034612
- link still_chassis_assm: mass 1e-09 -> 1.23353; geometry collision box size=0.006 0.014 0.005; collision box size=0.006 0.014 0.005
- link wheel_assm: mass 1e-09 -> 0.0495; geometry collision cylinder length=0.006 radius=0.0069282; collision cylinder length=0.006 radius=0.0069282
- link wheel_assm_2: mass 1e-09 -> 0.0495; geometry collision cylinder length=0.006 radius=0.0069282; collision cylinder length=0.006 radius=0.0069282
- link wheel_assm_3: mass 1e-09 -> 0.0495; geometry collision cylinder length=0.006 radius=0.0069282; collision cylinder length=0.006 radius=0.0069282
- link wheel_assm_4: mass 1e-09 -> 0.0495; geometry collision cylinder length=0.006 radius=0.0069282; collision cylinder length=0.006 radius=0.0069282
Joints:
- removed joint rplidar_a1_head_detector_ipt_fixed
- removed joint rplidar_a1_head_detector_mount_ipt_fixed
- removed joint rplidar_a1_head_head_ipt_fixed
- removed joint rplidar_a1_head_laser_ipt_fixed
- removed joint rplidar_a1_head_laser_mount_ipt_fixed
- removed joint rplidar_a1_head_woodscrews_gb_type136_m2x6_n_ipt_3_fixed
- removed joint rplidar_a1_head_woodscrews_gb_type136_m2x6_n_ipt_4_fixed
- removed joint rplidar_a1_head_woodscrews_gb_type136_m2x6_n_ipt_5_fixed
- removed joint still_chassis_assm_base_ipt_fixed
- removed joint still_chassis_assm_bn_3318_3664352_hex_stand_off_m2_5x16_10_fixed
- removed joint still_chassis_assm_bn_3318_3664352_hex_stand_off_m2_5x16_11_fixed
- removed joint still_chassis_assm_bn_3318_3664352_hex_stand_off_m2_5x16_12_fixed
- removed joint still_chassis_assm_bn_3318_3664352_hex_stand_off_m2_5x16_2_fixed
- removed joint still_chassis_assm_bn_3318_3664352_hex_stand_off_m2_5x16_3_fixed
- removed joint still_chassis_assm_bn_3318_3664352_hex_stand_off_m2_5x16_4_fixed
- removed joint still_chassis_assm_bn_3318_3664352_hex_stand_off_m2_5x16_5_fixed
- removed joint still_chassis_assm_bn_3318_3664352_hex_stand_off_m2_5x16_6_fixed
- removed joint still_chassis_assm_bn_3318_3664352_hex_stand_off_m2_5x16_7_fixed
- removed joint still_chassis_assm_bn_3318_3664352_hex_stand_off_m2_5x16_8_fixed
- removed joint still_chassis_assm_bn_3318_3664352_hex_stand_off_m2_5x16_9_fixed
- removed joint still_chassis_assm_bn_3318_3664352_hex_stand_off_m2_5x16_fixed
- removed joint still_chassis_assm_chassis_plate_2_fixed
- removed joint still_chassis_assm_chassis_plate_fixed
- removed joint still_chassis_assm_connector_1_25_3pin_ipt_fixed
- removed joint still_chassis_assm_connector_1_25_4pin_ipt_fixed
- removed joint still_chassis_assm_head_base_ipt_fixed
- removed joint still_chassis_assm_motherboard_ipt_fixed
- removed joint still_chassis_assm_motor_board_ipt_fixed
- removed joint still_chassis_assm_motor_bracket_md520_2_fixed
- removed joint still_chassis_assm_motor_bracket_md520_3_fixed
- removed joint still_chassis_assm_motor_bracket_md520_4_fixed
- removed joint still_chassis_assm_motor_bracket_md520_fixed
- removed joint still_chassis_assm_motor_ipt_fixed
- removed joint still_chassis_assm_motor_md520z30_12v_2_fixed
- removed joint still_chassis_assm_motor_md520z30_12v_3_fixed
- removed joint still_chassis_assm_motor_md520z30_12v_4_fixed
- removed joint still_chassis_assm_motor_md520z30_12v_fixed
- removed joint still_chassis_assm_rubber_ipt_fixed
- removed joint still_chassis_assm_spacer_m3_5_60_2_fixed
- removed joint still_chassis_assm_spacer_m3_5_60_3_fixed
- removed joint still_chassis_assm_spacer_m3_5_60_4_fixed
- removed joint still_chassis_assm_spacer_m3_5_60_5_fixed
- removed joint still_chassis_assm_spacer_m3_5_60_6_fixed
- removed joint still_chassis_assm_spacer_m3_5_60_fixed
- removed joint still_chassis_assm_wheel_ipt_fixed
- removed joint still_chassis_assm_woodscrews_gb_type136_m2x6_n_ipt_2_fixed
- removed joint still_chassis_assm_woodscrews_gb_type136_m2x6_n_ipt_fixed
- removed joint wheel_assm_2_hex_coupler_6mm_2_fixed
- removed joint wheel_assm_2_wheel_2_fixed
- removed joint wheel_assm_3_hex_coupler_6mm_3_fixed
- removed joint wheel_assm_3_wheel_3_fixed
- removed joint wheel_assm_4_hex_coupler_6mm_4_fixed
- removed joint wheel_assm_4_wheel_4_fixed
- removed joint wheel_assm_hex_coupler_6mm_fixed
- removed joint wheel_assm_wheel_fixed

Commit message: make lidar fixed joint

File: src/ballbot_description/onshape/ballbot_generated/robot.urdf (robot description, URDF)
Before this commit: robot ballbot_generated, 7 links, 6 joints
Joints:
- joint front_right_wheel_speed: origin xyz=0.0680211 -0.0776141 -0.0305 rpy=-1.5708 -1.26838 -1.05043e-15 -> xyz=0.0680211 -0.0776141 -0.0305 rpy=1.5708 -1.24974 -3.14159
- joint lidar: limit lower=-3.141592653589793 upper=3.141592653589793 effort=10 velocity=10 -> effort=10 velocity=10; origin xyz=0.0855211 0.000385868 0.12876 rpy=-3.14159 6.81317e-14 1.05236 -> xyz=0.0855211 0.000385868 0.1195 rpy=-3.14159 -4.57342e-14 1.72878; type revolute -> fixed

File: src/ballbot_description/urdf/ballbot.urdf (robot description, URDF)
Before this commit: robot ballbot_generated, 7 links, 6 joints
Joints:
- joint front_right_wheel_speed: origin xyz=0.0680211 -0.0776141 -0.0305 rpy=-1.5708 -1.26838 -1.05043e-15 -> xyz=0.0680211 -0.0776141 -0.0305 rpy=1.5708 -1.24974 -3.14159
- joint lidar: limit lower=-3.141592653589793 upper=3.141592653589793 effort=10 velocity=10 -> effort=10 velocity=10; origin xyz=0.0855211 0.000385868 0.12876 rpy=-3.14159 6.81317e-14 1.05236 -> xyz=0.0855211 0.000385868 0.1195 rpy=-3.14159 -4.57342e-14 1.72878; type revolute -> fixed

Commit message: physical imu link shown in rviz and gazebo

File: src/ballbot_description/onshape/ballbot_generated/robot.urdf (robot description, URDF)
Before this commit: robot ballbot_generated, 7 links, 6 joints
Links:
- added link mpu_9250, mass 0.00102531; collision cylinder length=0.002 radius=0.0005; collision cylinder length=0.002 radius=0.0005
- link still_chassis_assm: mass 1.23353 -> 1.23648; geometry collision box size=0.006 0.014 0.005; collision box size=0.006 0.014 0.005
Joints:
- added joint imu: type fixed, parent still_chassis_assm, child mpu_9250, origin xyz=-0.108479 0.0103859 0.005 rpy=-3.14159 -0 -3.14159, axis 0 0 1, limit effort=10 velocity=10

File: src/ballbot_description/urdf/ballbot.urdf (robot description, URDF)
Before this commit: robot ballbot_generated, 7 links, 6 joints
Links:
- added link mpu_9250, mass 0.00102531; collision cylinder length=0.002 radius=0.0005; collision cylinder length=0.002 radius=0.0005
- link still_chassis_assm: mass 1.23353 -> 1.23648; geometry collision box size=0.006 0.014 0.005; collision box size=0.006 0.014 0.005
Joints:
- added joint imu: type fixed, parent still_chassis_assm, child mpu_9250, origin xyz=-0.108479 0.0103859 0.005 rpy=-3.14159 -0 -3.14159, axis 0 0 1, limit effort=10 velocity=10

Commit message: add webcam CAD and pureshapes

File: src/ballbot_description/onshape/ballbot_generated/robot.urdf (robot description, URDF)
Before this commit: robot ballbot_generated, 8 links, 7 joints
Links:
- added link webcam, mass 0.019904; collision box size=0.079734 0.033688 0.024; collision cylinder length=0.017 radius=0.006
- link still_chassis_assm: mass 1.23648 -> 1.27612; geometry collision box size=0.006 0.014 0.005; collision box size=0.006 0.014 0.005
Joints:
- added joint webcam: type revolute, parent still_chassis_assm, child webcam, origin xyz=0.114021 -0.00486413 0.0545333 rpy=-1.5708 -1.5708 0, axis 0 0 1, limit lower=-3.141592653589793 upper=3.141592653589793 effort=10 velocity=10

File: src/ballbot_description/urdf/ballbot.urdf (robot description, URDF)
Before this commit: robot ballbot_generated, 8 links, 7 joints
Links:
- added link webcam, mass 0.019904; collision box size=0.079734 0.033688 0.024; collision cylinder length=0.017 radius=0.006
- link still_chassis_assm: mass 1.23648 -> 1.27612; geometry collision box size=0.006 0.014 0.005; collision box size=0.006 0.014 0.005
Joints:
- added joint webcam: type revolute, parent still_chassis_assm, child webcam, origin xyz=0.114021 -0.00486413 0.0545333 rpy=-1.5708 -1.5708 0, axis 0 0 1, limit lower=-3.141592653589793 upper=3.141592653589793 effort=10 velocity=10

Commit message: camera working but image upside down in rviz

File: src/ballbot_description/onshape/ballbot_generated/robot.urdf (robot description, URDF)
Before this commit: robot ballbot_generated, 9 links, 8 joints
Links:
- removed link webcam
- added link camera_link_optical
- added link camera_sensor_mount
- added link webcam_glass, mass 0.00160321; visual mesh filename=package://assets/webcam_glass.stl
- link still_chassis_assm: mass 1.27612 -> 1.29443; geometry collision box size=0.006 0.014 0.005; collision box size=0.006 0.014 0.005
Joints:
- added joint camera_optical_joint: type fixed, parent camera_sensor_mount, child camera_link_optical, origin xyz=0 0 0 rpy=-1.57 1.5708 -1.57
- added joint webcam_to_sensor_mount_joint: type fixed, parent webcam_glass, child camera_sensor_mount, origin xyz=0 0 0 rpy=0 1.5708 0
- joint webcam: child webcam -> webcam_glass; limit lower=-3.141592653589793 upper=3.141592653589793 effort=10 velocity=10 -> effort=10 velocity=10; origin xyz=0.114021 -0.00486413 0.0545333 rpy=-1.5708 -1.5708 0 -> xyz=0.152521 0.00263587 0.0545333 rpy=3.14159 1.5708 0; type revolute -> fixed

File: src/ballbot_description/urdf/ballbot.urdf (robot description, URDF)
Before this commit: robot ballbot_generated, 9 links, 8 joints
Links:
- removed link webcam
- added link camera_link_optical
- added link camera_sensor_mount
- added link webcam_glass, mass 0.00160321; visual mesh filename=package://ballbot_description/meshes/webcam_glass.stl
- link still_chassis_assm: mass 1.27612 -> 1.29443; geometry collision box size=0.006 0.014 0.005; collision box size=0.006 0.014 0.005
Joints:
- added joint camera_optical_joint: type fixed, parent camera_sensor_mount, child camera_link_optical, origin xyz=0 0 0 rpy=-1.5708 0 -1.5708
- added joint webcam_to_sensor_mount_joint: type fixed, parent webcam_glass, child camera_sensor_mount, origin xyz=0 0 0 rpy=0 1.5708 0
- joint webcam: child webcam -> webcam_glass; limit lower=-3.141592653589793 upper=3.141592653589793 effort=10 velocity=10 -> effort=10 velocity=10; origin xyz=0.114021 -0.00486413 0.0545333 rpy=-1.5708 -1.5708 0 -> xyz=0.152521 0.00263587 0.0545333 rpy=3.14159 1.5708 0; type revolute -> fixed

Commit message: fix camera orientation

File: src/ballbot_description/onshape/ballbot_generated/robot.urdf (robot description, URDF)
Before this commit: robot ballbot_generated, 11 links, 10 joints
Joints:
- joint camera_optical_joint: origin xyz=0 0 0 rpy=-1.57 1.5708 -1.57 -> xyz=0 0 0 rpy=-1.5708 0 -1.5708
- joint webcam_to_sensor_mount_joint: origin xyz=0 0 0 rpy=0 1.5708 0 -> xyz=0 0 0 rpy=3.14159 1.5708 0

File: src/ballbot_description/urdf/ballbot.urdf (robot description, URDF)
Before this commit: robot ballbot_generated, 11 links, 10 joints
Joints:
- joint webcam_to_sensor_mount_joint: origin xyz=0 0 0 rpy=0 1.5708 0 -> xyz=0 0 0 rpy=3.14159 1.5708 0

Commit message: add dc-dc converter to urdf

File: src/ballbot_description/onshape/ballbot_generated/robot.urdf (robot description, URDF)
Before this commit: robot ballbot_generated, 11 links, 10 joints
Links:
- link still_chassis_assm: mass 1.29443 -> 1.71089; geometry collision box size=0.006 0.014 0.005; collision box size=0.006 0.014 0.005
Joints:
- joint webcam: origin xyz=0.152521 0.00263587 0.0545333 rpy=3.14159 1.5708 0 -> xyz=0.158149 0.00263587 0.0556436 rpy=3.14159 1.5708 0

File: src/ballbot_description/urdf/ballbot.urdf (robot description, URDF)
Before this commit: robot ballbot_generated, 11 links, 10 joints
Links:
- link still_chassis_assm: mass 1.29443 -> 1.71089; geometry collision box size=0.006 0.014 0.005; collision box size=0.006 0.014 0.005
Joints:
- joint webcam: origin xyz=0.152521 0.00263587 0.0545333 rpy=3.14159 1.5708 0 -> xyz=0.158149 0.00263587 0.0556436 rpy=3.14159 1.5708 0
