Commit message: complete CAD model

File: src/ballbot_description/onshape/ballbot_generated/robot.urdf (robot description, URDF)
Before this commit: robot ballbot_generated, 11 links, 10 joints
Links:
- added link cam_3_lens_front, mass 2.21049e-06; visual mesh filename=package://assets/cam_3_lens_front.stl
- link mpu_9250: mass 0.00102531 -> 0.00152565; geometry visual mesh filename=package://assets/mpu_9250.stl; visual mesh filename=package://assets/mpu_9250_headers.stl
- link rplidar_a1_head: mass 0.0241835 -> 0.0241839; geometry visual mesh filename=package://assets/rplidar_a1_head.stl
- link still_chassis_assm: mass 1.71089 -> 2.02918; geometry collision box size=0.006 0.014 0.005; collision box size=0.006 0.014 0.005
Joints:
- added joint camera_module_lens: type fixed, parent still_chassis_assm, child cam_3_lens_front, origin xyz=0.103041 8.68467e-07 0.090095 rpy=3.14159 1.5708 0, axis 0 0 1, limit effort=10 velocity=10
- joint front_right_wheel_speed: origin xyz=0.0680211 -0.0776141 -0.0305 rpy=1.5708 -1.24974 -3.14159 -> xyz=0.0680211 -0.0776141 -0.0305 rpy=-1.5708 -1.53772 -1.03884e-14
- joint lidar: origin xyz=0.0855211 0.000385868 0.1195 rpy=-3.14159 -4.57342e-14 1.72878 -> xyz=0.0855211 0.000385868 0.1315 rpy=-3.14159 -1.87145e-13 3.07126
- joint rear_left_wheel_speed: origin xyz=-0.0804789 0.0783859 -0.0305 rpy=-1.5708 -0.366073 -6.32652e-16 -> xyz=-0.0804789 0.0783859 -0.0305 rpy=-1.5708 1.5708 0
- joint rear_right_wheel_speed: origin xyz=-0.0804789 -0.0776141 -0.0305 rpy=1.5708 1.46397 -3.14159 -> xyz=-0.0804789 -0.0776141 -0.0305 rpy=-1.5708 -1.53772 3.02617e-15

File: src/ballbot_description/urdf/ballbot.urdf (robot description, URDF)
Before this commit: robot ballbot_generated, 11 links, 10 joints
Links:
- added link cam_3_lens_front, mass 2.21049e-06; visual mesh filename=package://ballbot_description/meshes/cam_3_lens_front.stl
- link mpu_9250: mass 0.00102531 -> 0.00152565; geometry visual mesh filename=package://ballbot_description/meshes/mpu_9250.stl; visual mesh filename=package://ballbot_description/meshes/mpu_9250_headers.stl
- link rplidar_a1_head: mass 0.0241835 -> 0.0241839; geometry visual mesh filename=package://ballbot_description/meshes/rplidar_a1_head.stl
- link still_chassis_assm: mass 1.71089 -> 2.02918; geometry collision box size=0.006 0.014 0.005; collision box size=0.006 0.014 0.005
Joints:
- added joint camera_module_lens: type fixed, parent still_chassis_assm, child cam_3_lens_front, origin xyz=0.103041 8.68467e-07 0.090095 rpy=3.14159 1.5708 0, axis 0 0 1, limit effort=10 velocity=10
- joint front_right_wheel_speed: origin xyz=0.0680211 -0.0776141 -0.0305 rpy=1.5708 -1.24974 -3.14159 -> xyz=0.0680211 -0.0776141 -0.0305 rpy=-1.5708 -1.53772 -1.03884e-14
- joint lidar: origin xyz=0.0855211 0.000385868 0.1195 rpy=-3.14159 -4.57342e-14 1.72878 -> xyz=0.0855211 0.000385868 0.1315 rpy=-3.14159 -1.87145e-13 3.07126
- joint rear_left_wheel_speed: origin xyz=-0.0804789 0.0783859 -0.0305 rpy=-1.5708 -0.366073 -6.32652e-16 -> xyz=-0.0804789 0.0783859 -0.0305 rpy=-1.5708 1.5708 0
- joint rear_right_wheel_speed: origin xyz=-0.0804789 -0.0776141 -0.0305 rpy=1.5708 1.46397 -3.14159 -> xyz=-0.0804789 -0.0776141 -0.0305 rpy=-1.5708 -1.53772 3.02617e-15

Commit message: update to using onshape-to-robot master

File: src/ballbot_description/onshape/ballbot_generated/robot.urdf (robot description, URDF)
Before this commit: robot ballbot_generated, 12 links, 11 joints
Links:
- link still_chassis_assm: geometry collision box size=0.006 0.014 0.005; collision box size=0.006 0.014 0.005
- link wheel_assm: geometry collision cylinder length=0.006 radius=0.0069282; collision cylinder length=0.006 radius=0.0069282
- link wheel_assm_2: geometry collision cylinder length=0.006 radius=0.0069282; collision cylinder length=0.006 radius=0.0069282
- link wheel_assm_3: geometry collision cylinder length=0.006 radius=0.0069282; collision cylinder length=0.006 radius=0.0069282
- link wheel_assm_4: geometry collision cylinder length=0.006 radius=0.0069282; collision cylinder length=0.006 radius=0.0069282

File: src/ballbot_description/urdf/ballbot.urdf (robot description, URDF)
Before this commit: robot ballbot_generated, 12 links, 11 joints
Links:
- link still_chassis_assm: geometry collision box size=0.006 0.014 0.005; collision box size=0.006 0.014 0.005
- link wheel_assm: geometry collision cylinder length=0.006 radius=0.0069282; collision cylinder length=0.006 radius=0.0069282
- link wheel_assm_2: geometry collision cylinder length=0.006 radius=0.0069282; collision cylinder length=0.006 radius=0.0069282
- link wheel_assm_3: geometry collision cylinder length=0.006 radius=0.0069282; collision cylinder length=0.006 radius=0.0069282
- link wheel_assm_4: geometry collision cylinder length=0.006 radius=0.0069282; collision cylinder length=0.006 radius=0.0069282

Commit message: add base footprint

File: src/ballbot_description/onshape/ballbot_generated/robot.urdf (robot description, URDF)
Before this commit: robot ballbot_generated, 12 links, 11 joints
Links:
- added link base_footprint
- link base_link: mass 1e-09 -> None
Joints:
- added joint base_footprint_joint: type fixed, parent base_link, child base_footprint, origin xyz=0 0 -0.06449697 rpy=0 0 0

File: src/ballbot_description/urdf/ballbot.urdf (robot description, URDF)
Before this commit: robot ballbot_generated, 12 links, 11 joints
Links:
- added link base_footprint
- link base_link: mass 1e-09 -> None
Joints:
- added joint base_footprint_joint: type fixed, parent base_link, child base_footprint, origin xyz=0 0 -0.06449697 rpy=0 0 0

Commit message: make base_footprint parent of base_link

File: src/ballbot_description/onshape/ballbot_generated/robot.urdf (robot description, URDF)
Before this commit: robot ballbot_generated, 13 links, 12 joints
Joints:
- joint base_footprint_joint: child base_footprint -> base_link; origin xyz=0 0 -0.06449697 rpy=0 0 0 -> xyz=0 0 0.06449697 rpy=0 0 0; parent base_link -> base_footprint

File: src/ballbot_description/urdf/ballbot.urdf (robot description, URDF)
Before this commit: robot ballbot_generated, 13 links, 12 joints
Joints:
- joint base_footprint_joint: child base_footprint -> base_link; origin xyz=0 0 -0.06449697 rpy=0 0 0 -> xyz=0 0 0.06449697 rpy=0 0 0; parent base_link -> base_footprint

Commit message: try updating wheel joints

File: src/ballbot_description/onshape/ballbot_generated/robot.urdf (robot description, URDF)
Before this commit: robot ballbot_generated, 13 links, 12 joints
Joints:
- removed joint front_left_wheel_speed
- removed joint front_right_wheel_speed
- removed joint rear_left_wheel_speed
- removed joint rear_right_wheel_speed
- added joint front_left_wheel_joint_speed: type continuous, parent still_chassis_assm, child wheel_assm, origin xyz=0.0680211 0.0783859 -0.0305 rpy=-1.5708 -1.4446e-29 9.71445e-17, axis 0 0 1, limit effort=10 velocity=10
- added joint front_right_wheel_joint_speed: type continuous, parent still_chassis_assm, child wheel_assm_2, origin xyz=0.0680211 -0.0776141 -0.0305 rpy=-1.5708 -1.53772 -1.03884e-14, axis 0 0 1, limit effort=10 velocity=10
- added joint rear_left_wheel_joint_speed: type continuous, parent still_chassis_assm, child wheel_assm_3, origin xyz=-0.0804789 0.0783859 -0.0305 rpy=-1.5708 1.5708 0, axis 0 0 1, limit effort=10 velocity=10
- added joint rear_right_wheel_joint_speed: type continuous, parent still_chassis_assm, child wheel_assm_4, origin xyz=-0.0804789 -0.0776141 -0.0305 rpy=-1.5708 -1.53772 3.02617e-15, axis 0 0 1, limit effort=10 velocity=10

File: src/ballbot_description/urdf/ballbot.urdf (robot description, URDF)
Before this commit: robot ballbot_generated, 13 links, 12 joints
Joints:
- removed joint front_left_wheel_speed
- removed joint front_right_wheel_speed
- removed joint rear_left_wheel_speed
- removed joint rear_right_wheel_speed
- added joint front_left_wheel_joint_speed: type continuous, parent still_chassis_assm, child wheel_assm, origin xyz=0.0680211 0.0783859 -0.0305 rpy=-1.5708 -1.4446e-29 9.71445e-17, axis 0 0 1, limit effort=10 velocity=10
- added joint front_right_wheel_joint_speed: type continuous, parent still_chassis_assm, child wheel_assm_2, origin xyz=0.0680211 -0.0776141 -0.0305 rpy=-1.5708 -1.53772 -1.03884e-14, axis 0 0 1, limit effort=10 velocity=10
- added joint rear_left_wheel_joint_speed: type continuous, parent still_chassis_assm, child wheel_assm_3, origin xyz=-0.0804789 0.0783859 -0.0305 rpy=-1.5708 1.5708 0, axis 0 0 1, limit effort=10 velocity=10
- added joint rear_right_wheel_joint_speed: type continuous, parent still_chassis_assm, child wheel_assm_4, origin xyz=-0.0804789 -0.0776141 -0.0305 rpy=-1.5708 -1.53772 3.02617e-15, axis 0 0 1, limit effort=10 velocity=10

File: src/brobot_description/urdf/mech/wheel.urdf.xacro (robot description, xacro)
@@ -36,5 +36,5 @@
       </visual>
     </gazebo>
-    <joint name="${side}_wheel_joint" type="continuous">
+    <joint name="${side}_wheel_joint_speed" type="continuous">
       <axis xyz="0 1 0" />
       <parent link="base_link"/>
