Commit message: simplify config - post onshape move urdf and stl files

File: src/ballbot_description/urdf/ballbot.urdf (robot description, URDF)
Before this commit: robot ballbot_generated, 6 links, 5 joints
Links:
- link still_chassis_assm__configuration_default: geometry collision box size=0.006 0.014 0.005; collision box size=0.006 0.014 0.005
- link wheel_assm__configuration_default: geometry collision cylinder length=0.006 radius=0.0069282; collision cylinder length=0.006 radius=0.0069282
- link wheel_assm__configuration_default_2: geometry collision cylinder length=0.006 radius=0.0069282; collision cylinder length=0.006 radius=0.0069282
- link wheel_assm__configuration_default_3: geometry collision cylinder length=0.006 radius=0.0069282; collision cylinder length=0.006 radius=0.0069282
- link wheel_assm__configuration_default_4: geometry collision cylinder length=0.006 radius=0.0069282; collision cylinder length=0.006 radius=0.0069282

Commit message: fix(imu): publish sensor data in Z-up frame matching real chip
mpu_9250's link frame inherits onshape's part-local axes (Z-down), so
/imu/data was reporting accel.z = -9.79 m/s^2 stationary upright, and
the orientation quaternion was a 180-degree rotation. That's mirrored
from the physical chip on the real robot, which is mounted Z-up.

Add an imu_link child of mpu_9250 that cancels the parent joint's
(-pi, 0, -pi) flip, and move the gpu sensor onto imu_link with ROS 2
plugin syntax (the old <frameName>/<bodyName>/<rpyOffset> tags were
silently ignored by gazebo_ros_imu_sensor). The visual mesh stays on
mpu_9250 unchanged, so RViz/Gazebo rendering is unaffected.

Now publishes:
  frame_id          = imu_link  (matches firmware imu_interface.h:56)
  linear_accel.z    = +9.80     (Z-up, REP-145)
  orientation       ~ identity

File: src/ballbot_description/urdf/ballbot.urdf (robot description, URDF)
Before this commit: robot ballbot_generated, 13 links, 12 joints
Links:
- added link imu_link
Joints:
- added joint imu_link_joint: type fixed, parent mpu_9250, child imu_link, origin xyz=0 0 0 rpy=3.14159 0 3.14159
